File: _saved_photodiode_pcb.sch (KiCad schematic (older format))
At the start: 14 parts, among them P1 CONN_01X04, U1 LTC2461, U4 OPA381

Commit message: Update footprint
Parts:
- D1: renamed from D?; footprint (none) -> jnod_footprints:TO-5-3
Changed lines of the file:
@@
 $EndComp
 $Comp
-L GND #PWR5
+L GND #PWR01
 U 1 1 569AD39F
 P 4400 3050
-F 0 "#PWR5" H 4400 2800 50  0001 C CNN
+F 0 "#PWR01" H 4400 2800 50  0001 C CNN
 F 1 "GND" H 4400 2900 50  0000 C CNN
 F 2 "" H 4400 3050 50  0000 C CNN
@@
 $EndComp
 $Comp
-L GND #PWR4
+L GND #PWR02
 U 1 1 569AE178
 P 4400 2600
-F 0 "#PWR4" H 4400 2350 50  0001 C CNN
+F 0 "#PWR02" H 4400 2350 50  0001 C CNN
 F 1 "GND" H 4400 2450 50  0000 C CNN
 F 2 "" H 4400 2600 50  0000 C CNN
@@
 $EndComp
 $Comp
-L VCC #PWR14
+L VCC #PWR03
 U 1 1 569AF392
 P 7000 4200
-F 0 "#PWR14" H 7000 4050 50  0001 C CNN
+F 0 "#PWR03" H 7000 4050 50  0001 C CNN
 F 1 "VCC" H 7000 4350 50  0000 C CNN
 F 2 "" H 7000 4200 50  0000 C CNN
@@
 $EndComp
 $Comp
-L GND #PWR15
+L GND #PWR04
 U 1 1 569AF4AF
 P 7000 4500
-F 0 "#PWR15" H 7000 4250 50  0001 C CNN
+F 0 "#PWR04" H 7000 4250 50  0001 C CNN
 F 1 "GND" H 7000 4350 50  0000 C CNN
 F 2 "" H 7000 4500 50  0000 C CNN
@@
 $EndComp
 $Comp
-L GND #PWR6
+L GND #PWR05
 U 1 1 569AF99E
 P 5500 4450
-F 0 "#PWR6" H 5500 4200 50  0001 C CNN
+F 0 "#PWR05" H 5500 4200 50  0001 C CNN
 F 1 "GND" H 5500 4300 50  0000 C CNN
 F 2 "" H 5500 4450 50  0000 C CNN
@@
 $EndComp
 $Comp
-L VCC #PWR2
+L VCC #PWR06
 U 1 1 569AFDE2
 P 4200 2750
-F 0 "#PWR2" H 4200 2600 50  0001 C CNN
+F 0 "#PWR06" H 4200 2600 50  0001 C CNN
 F 1 "VCC" H 4200 2900 50  0000 C CNN
 F 2 "" H 4200 2750 50  0000 C CNN
@@
 $EndComp
 $Comp
-L GND #PWR8
+L GND #PWR07
 U 1 1 569B1CCA
 P 5850 4500
-F 0 "#PWR8" H 5850 4250 50  0001 C CNN
+F 0 "#PWR07" H 5850 4250 50  0001 C CNN
 F 1 "GND" H 5850 4350 50  0000 C CNN
 F 2 "" H 5850 4500 50  0000 C CNN
@@
 $EndComp
 $Comp
-L GND #PWR13
+L GND #PWR08
 U 1 1 569B3249
 P 6750 3550
-F 0 "#PWR13" H 6750 3300 50  0001 C CNN
+F 0 "#PWR08" H 6750 3300 50  0001 C CNN
 F 1 "GND" H 6750 3400 50  0000 C CNN
 F 2 "" H 6750 3550 50  0000 C CNN
@@
 $EndComp
 $Comp
-L GND #PWR1
+L GND #PWR09
 U 1 1 569C0022
 P 4000 3550
-F 0 "#PWR1" H 4000 3300 50  0001 C CNN
+F 0 "#PWR09" H 4000 3300 50  0001 C CNN
 F 1 "GND" H 4000 3400 50  0000 C CNN
 F 2 "" H 4000 3550 50  0000 C CNN
@@
 $EndComp
 $Comp
-L GND #PWR12
+L GND #PWR010
 U 1 1 569C085F
 P 6400 3700
-F 0 "#PWR12" H 6400 3450 50  0001 C CNN
+F 0 "#PWR010" H 6400 3450 50  0001 C CNN
 F 1 "GND" H 6400 3550 50  0000 C CNN
 F 2 "" H 6400 3700 50  0000 C CNN
@@
 $EndComp
 $Comp
-L GND #PWR7
+L GND #PWR011
 U 1 1 569C0987
 P 5700 4050
-F 0 "#PWR7" H 5700 3800 50  0001 C CNN
+F 0 "#PWR011" H 5700 3800 50  0001 C CNN
 F 1 "GND" H 5700 3900 50  0000 C CNN
 F 2 "" H 5700 4050 50  0000 C CNN
@@
 $EndComp
 $Comp
-L VCC #PWR10
+L VCC #PWR012
 U 1 1 569C1370
 P 6200 3450
-F 0 "#PWR10" H 6200 3300 50  0001 C CNN
+F 0 "#PWR012" H 6200 3300 50  0001 C CNN
 F 1 "VCC" H 6200 3600 50  0000 C CNN
 F 2 "" H 6200 3450 50  0000 C CNN
@@
 $EndComp
 $Comp
-L GND #PWR3
+L GND #PWR013
 U 1 1 569C17EB
 P 4350 3850
-F 0 "#PWR3" H 4350 3600 50  0001 C CNN
+F 0 "#PWR013" H 4350 3600 50  0001 C CNN
 F 1 "GND" H 4350 3700 50  0000 C CNN
 F 2 "" H 4350 3850 50  0000 C CNN
@@
 SCL
 $Comp
-L PWR_FLAG #FLG1
+L PWR_FLAG #FLG014
 U 1 1 56AD25FD
 P 5900 2350
-F 0 "#FLG1" H 5900 2445 50  0001 C CNN
+F 0 "#FLG014" H 5900 2445 50  0001 C CNN
 F 1 "PWR_FLAG" H 5900 2530 50  0000 C CNN
 F 2 "" H 5900 2350 50  0000 C CNN
@@
 $EndComp
 $Comp
-L PWR_FLAG #FLG2
+L PWR_FLAG #FLG015
 U 1 1 56AD2653
 P 6300 2350
-F 0 "#FLG2" H 6300 2445 50  0001 C CNN
+F 0 "#FLG015" H 6300 2445 50  0001 C CNN
 F 1 "PWR_FLAG" H 6300 2530 50  0000 C CNN
 F 2 "" H 6300 2350 50  0000 C CNN
@@
 $EndComp
 $Comp
-L VCC #PWR9
+L VCC #PWR016
 U 1 1 56AD2682
 P 5900 2450
-F 0 "#PWR9" H 5900 2300 50  0001 C CNN
+F 0 "#PWR016" H 5900 2300 50  0001 C CNN
 F 1 "VCC" H 5900 2600 50  0000 C CNN
 F 2 "" H 5900 2450 50  0000 C CNN
@@
 	5900 2350 5900 2450
 $Comp
-L GND #PWR11
+L GND #PWR017
 U 1 1 56AD2722
 P 6300 2450
-F 0 "#PWR11" H 6300 2200 50  0001 C CNN
+F 0 "#PWR017" H 6300 2200 50  0001 C CNN
 F 1 "GND" H 6300 2300 50  0000 C CNN
 F 2 "" H 6300 2450 50  0000 C CNN
@@
 NoConn ~ 6400 5150
 $Comp
-L photodiode_asc D?
+L photodiode_asc D1
 U 1 1 56DC95DD
 P 5100 4300
-F 0 "D?" H 5100 4400 60  0000 C CNN
+F 0 "D1" H 5100 4400 60  0000 C CNN
 F 1 "photodiode_asc" H 5100 4300 60  0000 C CNN
-F 2 "" H 5100 4300 60  0000 C CNN
+F 2 "jnod_footprints:TO-5-3" H 5100 4300 60  0001 C CNN
 F 3 "" H 5100 4300 60  0000 C CNN
 	1    5100 4300
